Commit message: Added Lidar model

File: description/robot.urdf.xacro (robot description, xacro)
@@ -2,3 +2,4 @@
 <robot xmlns:xacro="http://www.ros.org/wiki/xacro"  name="robot">
     <xacro:include filename="robot_core.xacro" />
+    <xacro:include filename="lidar.xacro" />
 </robot>

File: description/robot_core.xacro (robot description, xacro)
@@ -13,4 +13,7 @@
     <material name="black">
         <color rgba="0 0 0 1" />
+    </material>
+    <material name="red">
+        <color rgba="1 0 0 1" />
     </material>
     <!--BASE LINK-->
@@ -41,4 +44,7 @@
         </xacro:inertial_box>
     </link>
+    <gazebo reference="chassis">
+        <material>Gazebo/White</material>
+    </gazebo>
     <!--LEFT BACK WHEEL LINK-->
     <joint name="left_back_wheel_joint" type="continuous">
@@ -64,4 +70,7 @@
         </xacro:inertial_cylinder>
     </link>
+    <gazebo reference="left_back_wheel">
+        <material>Gazebo/Blue</material>
+    </gazebo>
     <!--RIGHT BACK WHEEL LINK-->
     <joint name="right_back_wheel_joint" type="continuous">
@@ -87,4 +96,7 @@
         </xacro:inertial_cylinder>
     </link>
+    <gazebo reference="right_back_wheel">
+        <material>Gazebo/Blue</material>
+    </gazebo>
     <!--LEFT FRONT WHEEL LINK-->
     <joint name="left_front_wheel_joint" type="continuous">
@@ -110,4 +122,7 @@
         </xacro:inertial_cylinder>
     </link>
+    <gazebo reference="left_front_wheel">
+        <material>Gazebo/Blue</material>
+    </gazebo>
     <!--RIGHT FRONT WHEEL LINK-->
     <joint name="right_front_wheel_joint" type="continuous">
@@ -133,3 +148,6 @@
         </xacro:inertial_cylinder>
     </link>
+    <gazebo reference="right_front_wheel">
+        <material>Gazebo/Blue</material>
+    </gazebo>
 </robot>
